File: Pathfinder efidget.kicad_pcb (KiCad board)
At the start: 2 copper layers, 63.5 x 72 mm, 19 parts, among them SW1 SW_Push, SW2 SW_Push, SW3 SW_Push, SW4 SW_Push, U1 MOUDLE-SEEEDUINO-XIAO

Commit message: Add files via upload
Parts:
- moved U1 2.99 mm to (122.0, 119.4)
Routing:
- net Led3: track 36.3 -> 41.8 mm
- net Button3: track 60.8 -> 66.2 mm
- net Button4: track 34.6 -> 38.6 mm
- net Led4: track 42.5 -> 45.5 mm
- net Led2: track 50.5 -> 52.5 mm
- net Button1: track 70.3 -> 72.1 mm
- net Button2: track 65.4 -> 63.8 mm
- net Led1: track 63.3 -> 64.5 mm
- net GND: track 151.8 -> 153.1 mm
- net Buzzer: track 22.3 -> 21.1 mm
Changed lines of the file:
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@@
 			(outputformat 1)
 			(mirror no)
-			(drillshape 1)
+			(drillshape 0)
 			(scaleselection 1)
-			(outputdirectory "")
+			(outputdirectory "Gerber/")
 		)
 	)
@@
 	(footprint "footprints:XIAO-Generic-Hybrid-14P-2.54-21X17.8MM"
 		(layer "F.Cu")
-		(at 122 116.3895 180)
+		(at 122 119.38 180)
 		(property "Reference" "U1"
 			(at 0 2.54 0)
@@
 	)
 	(segment
-		(start 99.3905 111.3095)
-		(end 114.375 111.3095)
+		(start 114.375 114.3)
+		(end 96.4 114.3)
 		(width 0.2)
 		(layer "F.Cu")
@@
 	(segment
 		(start 94.2 116.5)
-		(end 99.3905 111.3095)
+		(end 96.4 114.3)
 		(width 0.2)
 		(layer "F.Cu")
@@
 	)
 	(segment
+		(start 101.8 116.5)
+		(end 109.76 124.46)
+		(width 0.2)
+		(layer "B.Cu")
+		(net 2)
+	)
+	(segment
 		(start 96.77 68.46)
 		(end 115.77 68.46)
@@
 	)
 	(segment
-		(start 101.8 116.5)
-		(end 106.7695 121.4695)
-		(width 0.2)
-		(layer "B.Cu")
-		(net 2)
-	)
-	(segment
 		(start 96.77 68.46)
 		(end 96.77 87.46)
@@
 	)
 	(segment
-		(start 106.7695 121.4695)
-		(end 114.375 121.4695)
+		(start 109.76 124.46)
+		(end 114.375 124.46)
 		(width 0.2)
 		(layer "B.Cu")
@@
 	)
 	(segment
-		(start 134 113.5)
-		(end 129.9745 113.5)
-		(width 0.2)
-		(layer "F.Cu")
-		(net 7)
-	)
-	(segment
 		(start 150 68.96)
 		(end 150 97.5)
@@
 	)
 	(segment
-		(start 129.9745 113.5)
-		(end 129.625 113.8495)
+		(start 134 113.50276)
+		(end 130.66276 116.84)
 		(width 0.2)
 		(layer "F.Cu")
@@
 	)
 	(segment
+		(start 130.66276 116.84)
+		(end 129.625 116.84)
+		(width 0.2)
+		(layer "F.Cu")
+		(net 7)
+	)
+	(segment
 		(start 134.5 106)
 		(end 134.5 113)
@@
 	)
 	(segment
+		(start 134 113.5)
+		(end 134 113.50276)
+		(width 0.2)
+		(layer "F.Cu")
+		(net 7)
+	)
+	(segment
 		(start 134.5 113)
 		(end 134 113.5)
@@
 	)
 	(segment
-		(start 147.61 75.476894)
-		(end 149.5 77.366894)
+		(start 141 98.5)
+		(end 133.5 106)
 		(width 0.2)
 		(layer "F.Cu")
@@
 	)
 	(segment
-		(start 148 98.5)
-		(end 141 98.5)
+		(start 133.5 106)
+		(end 133.5 111.46276)
 		(width 0.2)
 		(layer "F.Cu")
@@
 	)
 	(segment
-		(start 149.5 77.366894)
-		(end 149.5 97)
+		(start 130.66276 114.3)
+		(end 129.625 114.3)
 		(width 0.2)
 		(layer "F.Cu")
@@
 	)
 	(segment
-		(start 141 98.5)
-		(end 133.5 106)
+		(start 149.5 77.366894)
+		(end 149.5 97)
 		(width 0.2)
 		(layer "F.Cu")
@@
 	)
 	(segment
-		(start 133.5 110)
-		(end 132.1905 111.3095)
+		(start 148 98.5)
+		(end 141 98.5)
 		(width 0.2)
 		(layer "F.Cu")
@@
 	)
 	(segment
-		(start 132.1905 111.3095)
-		(end 129.625 111.3095)
+		(start 133.5 111.46276)
+		(end 130.66276 114.3)
 		(width 0.2)
 		(layer "F.Cu")
@@
 	)
 	(segment
-		(start 133.5 106)
-		(end 133.5 110)
+		(start 147.61 75.476894)
+		(end 149.5 77.366894)
 		(width 0.2)
 		(layer "F.Cu")
@@
 	)
 	(segment
+		(start 129.625 108.7695)
+		(end 129.625 111.76)
+		(width 0.2)
+		(layer "F.Cu")
+		(net 9)
+	)
+	(segment
 		(start 149 86.029788)
 		(end 149 96.5)
@@
 	)
 	(segment
+		(start 132.1905 111.3095)
+		(end 129.625 111.3095)
+		(width 0.2)
+		(layer "F.Cu")
+		(net 9)
+	)
+	(segment
 		(start 140.3945 98)
 		(end 147.5 98)
@@
 	)
 	(segment
-		(start 120.5 100)
-		(end 114.375 106.125)
+		(start 148 95.104682)
+		(end 148 98)
 		(width 0.2)
 		(layer "B.Cu")
@@
 	)
 	(segment
-		(start 146 100)
-		(end 120.5 100)
+		(start 114.375 106.125)
+		(end 114.375 111.76)
 		(width 0.2)
 		(layer "B.Cu")
@@
 	)
 	(segment
-		(start 148 95.104682)
-		(end 148 98)
+		(start 146 100)
+		(end 120.5 100)
 		(width 0.2)
 		(layer "B.Cu")
@@
 	)
 	(segment
-		(start 114.375 106.125)
-		(end 114.375 108.7695)
+		(start 148 98)
+		(end 146 100)
 		(width 0.2)
 		(layer "B.Cu")
@@
 	)
 	(segment
-		(start 148 98)
-		(end 146 100)
+		(start 120.5 100)
+		(end 114.375 106.125)
 		(width 0.2)
 		(layer "B.Cu")
@@
 	)
 	(segment
-		(start 118.606184 92.351)
-		(end 118.606184 115.106184)
+		(start 118.606184 115.106184)
+		(end 129.625 126.125)
 		(width 0.2)
 		(layer "F.Cu")
@@
 	)
 	(segment
-		(start 118.606184 115.106184)
-		(end 127.5095 124.0095)
+		(start 103.12 76.864816)
+		(end 118.606184 92.351)
 		(width 0.2)
 		(layer "F.Cu")
@@
 	)
 	(segment
-		(start 103.12 76.864816)
-		(end 118.606184 92.351)
+		(start 129.625 126.125)
+		(end 129.625 127)
 		(width 0.2)
 		(layer "F.Cu")
@@
 	)
 	(segment
-		(start 103.12 65.92)
-		(end 103.12 76.864816)
+		(start 118.606184 92.351)
+		(end 118.606184 115.106184)
 		(width 0.2)
 		(layer "F.Cu")
@@
 	)
 	(segment
-		(start 127.5095 124.0095)
-		(end 129.625 124.0095)
+		(start 103.12 65.92)
+		(end 103.12 76.864816)
 		(width 0.2)
 		(layer "F.Cu")
@@
 	)
 	(segment
-		(start 133.5 123)
-		(end 131.9695 121.4695)
+		(start 132.676 128.151)
+		(end 128.651 128.151)
 		(width 0.2)
 		(layer "F.Cu")
@@
 	)
 	(segment
-		(start 103.12 84.92)
-		(end 117 98.8)
+		(start 128.651 128.151)
+		(end 117 116.5)
 		(width 0.2)
 		(layer "F.Cu")
@@
 	)
 	(segment
-		(start 131.9695 121.4695)
-		(end 129.625 121.4695)
+		(start 131.287 124.46)
+		(end 132.676 125.849)
 		(width 0.2)
 		(layer "F.Cu")
@@
 	)
 	(segment
-		(start 133.5 126.5)
-		(end 133.5 123)
+		(start 117 116.5)
+		(end 117 98.8)
 		(width 0.2)
 		(layer "F.Cu")
@@
 	)
 	(segment
-		(start 117 115.5)
-		(end 128 126.5)
+		(start 129.625 124.46)
+		(end 131.287 124.46)
 		(width 0.2)
 		(layer "F.Cu")
@@
 	)
 	(segment
-		(start 128 126.5)
-		(end 133.5 126.5)
+		(start 132.676 125.849)
+		(end 132.676 128.151)
 		(width 0.2)
 		(layer "F.Cu")
@@
 	(segment
 		(start 117 98.8)
-		(end 117 115.5)
+		(end 103.12 84.92)
 		(width 0.2)
 		(layer "F.Cu")
@@
 	)
 	(segment
-		(start 132.05176 115.2385)
-		(end 132.726 115.91274)
+		(start 129.625 121.92)
+		(end 130.66276 121.92)
 		(width 0.2)
 		(layer "F.Cu")
@@
 	)
 	(segment
-		(start 130.66276 118.9295)
-		(end 129.625 118.9295)
+		(start 128.524 117.31676)
+		(end 128.524 72.324)
 		(width 0.2)
 		(layer "F.Cu")
@@
 	)
 	(segment
-		(start 128.524 72.324)
-		(end 128.524 114.32626)
+		(start 131.81376 117.991)
+		(end 129.19824 117.991)
 		(width 0.2)
 		(layer "F.Cu")
@@
 	)
 	(segment
-		(start 128.524 114.32626)
-		(end 129.43624 115.2385)
+		(start 131.9695 121.4695)
+		(end 129.625 121.4695)
 		(width 0.2)
 		(layer "F.Cu")
@@
 	)
 	(segment
-		(start 122.12 65.92)
-		(end 128.524 72.324)
+		(start 132.726 119.85676)
+		(end 132.726 118.90324)
 		(width 0.2)
 		(layer "F.Cu")
@@
 	)
 	(segment
-		(start 132.726 115.91274)
-		(end 132.726 116.86626)
+		(start 129.19824 117.991)
+		(end 128.524 117.31676)
 		(width 0.2)
 		(layer "F.Cu")
@@
 	)
 	(segment
-		(start 132.726 116.86626)
-		(end 130.66276 118.9295)
+		(start 132.726 118.90324)
+		(end 131.81376 117.991)
+		(width 0.2)
+		(layer "F.Cu")
+		(net 13)
+	)
+	(segment
+		(start 128.524 72.324)
+		(end 122.12 65.92)
 		(width 0.2)
 		(layer "F.Cu")
@@
 	)
 	(segment
-		(start 129.43624 115.2385)
-		(end 132.05176 115.2385)
+		(start 130.66276 121.92)
+		(end 132.726 119.85676)
 		(width 0.2)
 		(layer "F.Cu")
@@
 	)
 	(segment
-		(start 122.12 84.92)
-		(end 122.12 108.8845)
+		(start 130.66276 118.9295)
+		(end 129.625 118.9295)
+		(width 0.2)
+		(layer "F.Cu")
+		(net 14)
+	)
+	(segment
+		(start 129.625 119.38)
+		(end 122.12 111.875)
 		(width 0.2)
 		(layer "F.Cu")
@@
 	)
 	(segment
-		(start 122.12 108.8845)
-		(end 129.625 116.3895)
+		(start 122.12 111.875)
+		(end 122.12 84.92)
 		(width 0.2)
 		(layer "F.Cu")
